Commit message: Added yolo, pose,tsk nodes

File: my_robot_task_api/urdf/gen3_final.urdf (robot description, URDF)
Before this commit: robot gen3_lite_gen3_lite_2f, 15 links, 14 joints
Links:
- added link camera_link, mass 0.01
Joints:
- added joint camera_joint: type fixed, parent base_link, child camera_link, origin xyz=0.25 0.0 1.20 rpy=0 1.57 0

Commit message: added robot publisher launch file & fixed optical frame

File: my_robot_task_api/urdf/gen3_final.urdf (robot description, URDF)
Before this commit: robot gen3_lite_gen3_lite_2f, 16 links, 15 joints
Links:
- added link rgbd_camera_frame
- added link rgbd_camera_optical_frame
Joints:
- added joint rgbd_camera_frame_joint: type fixed, parent camera_link, child rgbd_camera_frame, origin xyz=0 0 0 rpy=0 0 0
- added joint rgbd_camera_optical_joint: type fixed, parent rgbd_camera_frame, child rgbd_camera_optical_frame, origin xyz=0 0 0 rpy=-1.5708 0 -1.5708

Commit message: added models and yolo dataset

File: my_robot_task_api/urdf/gen3_final.urdf (robot description, URDF)
Before this commit: robot gen3_lite_gen3_lite_2f, 18 links, 17 joints
Joints:
- joint base_joint: origin xyz=0 0 0 rpy=0 0 0 -> xyz=0 0 0.30 rpy=0 0 0
- joint camera_joint: origin xyz=0.25 0.0 1.20 rpy=0 1.57 0 -> xyz=0.12 0.0 1.0 rpy=0 1.10 0

Commit message: Fixed Quaternions

File: my_robot_task_api/urdf/gen3_final.urdf (robot description, URDF)
Before this commit: robot gen3_lite_gen3_lite_2f, 18 links, 17 joints
Joints:
- joint base_joint: origin xyz=0 0 0.30 rpy=0 0 0 -> xyz=0 0 0 rpy=0 0 0

Commit message: Increased efforts of joints

File: my_robot_task_api/urdf/gen3_final.urdf (robot description, URDF)
Before this commit: robot gen3_lite_gen3_lite_2f, 18 links, 17 joints
Joints:
- joint joint_1: limit lower=-2.68 upper=2.68 effort=10 velocity=1.6 -> lower=-2.68 upper=2.68 effort=200 velocity=1.6
- joint joint_2: limit lower=-2.61 upper=2.61 effort=14 velocity=1.6 -> lower=-2.61 upper=2.61 effort=200 velocity=1.6
- joint joint_3: limit lower=-2.61 upper=2.61 effort=10 velocity=1.6 -> lower=-2.61 upper=2.61 effort=200 velocity=1.6
- joint joint_4: limit lower=-2.6 upper=2.6 effort=7 velocity=1.6 -> lower=-2.6 upper=2.6 effort=200 velocity=1.6
- joint joint_5: limit lower=-2.53 upper=2.53 effort=7 velocity=1.6 -> lower=-2.53 upper=2.53 effort=200 velocity=1.6
- joint joint_6: limit lower=-2.6 upper=2.6 effort=7 velocity=3.2 -> lower=-2.6 upper=2.6 effort=200 velocity=3.2
- joint right_finger_bottom_joint: limit lower=0.0 upper=0.85 effort=50 velocity=0.6 -> lower=0.0 upper=0.85 effort=100 velocity=0.6
